Commit message: Added improvements in dae

File: turtlebot3/turtlebot3_description/urdf/sensors.xacro (robot description, xacro)
@@ -6,5 +6,5 @@
                 <visual>
                     <geometry>
-                    <mesh filename="package://jetdog_description/meshes/sensors/rpi_camera_v2.dae"/>
+                    <mesh filename="package://turtlebot3_description/meshes/sensors/rpi_camera_v2.dae"/>
                     </geometry>
                     <material name="camera_link_material">
@@ -14,5 +14,5 @@
                 <collision>
                     <geometry>
-                    <mesh filename="package://jetdog_description/meshes/sensors/rpi_camera_v2.stl"/>
+                    <mesh filename="package://turtlebot3_description/meshes/sensors/rpi_camera_v2.stl"/>
                     </geometry>
                 </collision>
@@ -28,5 +28,5 @@
                 <visual>
                     <geometry>
-                    <mesh filename="package://jetdog_description/meshes/sensors/rpi_camera_v2_short.dae"/>
+                    <mesh filename="package://turtlebot3_description/meshes/sensors/rpi_camera_v2_short.dae"/>
                     </geometry>
                     <material name="camera_link_material">
@@ -36,5 +36,5 @@
                 <collision>
                     <geometry>
-                    <mesh filename="package://jetdog_description/meshes/sensors/rpi_camera_v2_short.stl"/>
+                    <mesh filename="package://turtlebot3_description/meshes/sensors/rpi_camera_v2_short.stl"/>
                     </geometry>
                 </collision>

File: turtlebot3/turtlebot3_description/urdf/turtlebot3_burger_rrl.urdf.xacro (robot description, xacro)
@@ -42,5 +42,5 @@
       <origin xyz="0 0 0" rpy="${M_PI*0.5} 0 0"/>
       <geometry>
-        <mesh filename="package://turtlebot3_description/meshes/wheels/left_tire.stl" scale="0.001 0.001 0.001"/>
+        <mesh filename="package://turtlebot3_description/meshes/wheels/left_tire.dae" scale="0.001 0.001 0.001"/>
       </geometry>
       <material name="dark"/>
@@ -70,5 +70,5 @@
       <origin xyz="0 0 0" rpy="${M_PI*0.5} 0 0"/>
       <geometry>
-        <mesh filename="package://turtlebot3_description/meshes/wheels/right_tire.stl" scale="0.001 0.001 0.001"/>
+        <mesh filename="package://turtlebot3_description/meshes/wheels/right_tire.dae" scale="0.001 0.001 0.001"/>
       </geometry>
       <material name="dark"/>
@@ -123,5 +123,5 @@
       <origin xyz="0 0 0.0" rpy="0 0 0"/>
       <geometry>
-        <mesh filename="package://turtlebot3_description/meshes/sensors/lds.stl" scale="0.001 0.001 0.001"/>
+        <mesh filename="package://turtlebot3_description/meshes/sensors/lds.dae" scale="0.001 0.001 0.001"/>
       </geometry>
       <material name="dark"/>

Commit message: Corrected camera pose

File: turtlebot3/turtlebot3_description/urdf/sensors.xacro (robot description, xacro)
@@ -47,5 +47,5 @@
         </xacro:if>
         <joint name="chassis_1_camera_link_fixing" type="fixed">
-            <origin xyz="-0.018139 0.000303 -0.01267" rpy="-1.57 0 3.14" />
+            <origin xyz="0.035 0.0 0.0614643" rpy="0 0 0" />
             <parent link="${parent}" />
             <child link="camera_link" />
@@ -72,5 +72,5 @@
         <xacro:if value="${version == 'long'}">
             <joint name="camera_frame_joint" type="fixed">
-                <origin xyz="0.0671392 0.0 0.0220048" rpy="0 0 0" />
+                <origin xyz="0.028402 0.000001 0.002402" rpy="0 0 0" />
                 <parent link="camera_link" />
                 <child link="camera_link_frame" />
@@ -80,5 +80,5 @@
         <xacro:if value="${version == 'short'}">
             <joint name="camera_frame_joint" type="fixed">
-                <origin xyz="0.0671392 0.0 0.0614643" rpy="0 0 0" />
+                <origin xyz="0.01 0.000001 0.002402" rpy="0 0 0" />
                 <parent link="camera_link" />
                 <child link="camera_link_frame" />
