Commit message: Added batery simulation for turtlebot3

File: turtlebot3/turtlebot3_description/urdf/turtlebot3_burger.gazebo.xacro (robot description, xacro)
@@ -22,5 +22,6 @@
   </gazebo>
   <gazebo reference="base_link">
-    <material>Gazebo/Grey</material>
+    <!--<material>Gazebo/DarkGrey</material>
+    -->
   </gazebo>
   <gazebo reference="wheel_left_link">
@@ -51,5 +52,5 @@
     <minDepth>0.001</minDepth>
     <maxVel>1.0</maxVel>
-    <material>Gazebo/Grey</material>
+    <material>Gazebo/DarkGrey</material>
   </gazebo>
   <gazebo>
@@ -86,5 +87,5 @@
       <visualize>$(arg imu_visual)</visualize>
     </sensor>
-    <material>Gazebo/Grey</material>
+    <material>Gazebo/DarkGrey</material>
   </gazebo>
   <gazebo reference="base_scan">
